File: Adjustable power supply/Adjustable power supply.kicad_pcb (KiCad board)
At the start: 2 copper layers, 57.8 x 36.8 mm, 9 parts, among them J1 Conn_01x02_Pin, J2 Conn_01x02_Pin, U1 LM317_TO-220

Commit message: test segment
test segment
Routing:
- net (no net): track 0.00 -> 3.96 mm
Changed lines of the file:
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@@
+	)
+	(segment
+		(start 142.24 62.23)
+		(end 142.24 60.96)
+		(width 0.2)
+		(layer "B.Cu")
+		(net 0)
+	)
+	(segment
+		(start 142.24 60.96)
+		(end 144.145 59.055)
+		(width 0.2)
+		(layer "B.Cu")
+		(net 0)
 	)
 	(segment

Commit message: reverse change
Routing:
- net (no net): track 3.96 -> 0.00 mm
Changed lines of the file:
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@@
 	)
 	(gr_text "Adjustable Power supply"
-		(at 101.6 74.93 -0)
+		(at 101.6 74.93 0)
 		(layer "B.Cu")
 		(effects
@@
 				(bold yes)
 			)
-			(justify left bottom mirror)
+			(justify left bottom)
 		)
 	)
@@
 	)
 	(segment
-		(start 142.24 62.23)
-		(end 142.24 60.96)
-		(width 0.2)
-		(layer "B.Cu")
-		(net 0)
-	)
-	(segment
-		(start 142.24 60.96)
-		(end 144.145 59.055)
-		(width 0.2)
-		(layer "B.Cu")
-		(net 0)
-	)
-	(segment
